File: CELL-MOUNT/CELL-MOUNT.kicad_pcb (KiCad board)
At the start: 2 copper layers, 120 x 220 mm, 52 parts

Commit message: Lock down before branch for projects
Other:
- outline, holes or cut-outs redrawn
Changed lines of the file:
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@@
   (general
     (thickness 1.6)
-    (drawings 108)
+    (drawings 84)
     (tracks 0)
     (zones 0)
@@
     (solder_mask_min_width 0.25)
     (aux_axis_origin 0 0)
-    (grid_origin 78 107.25)
+    (grid_origin 60 270)
     (visible_elements FFFFFF7F)
     (pcbplotparams
@@
     (pad 1 np_thru_hole circle (at 0 0) (size 4.3 4.3) (drill 4.3) (layers *.Cu *.Mask))
   )
-  (gr_arc (start 78 171) (end 79.5 171) (angle -180) (layer Edge.Cuts) (width 0.05))
-  (gr_line (start 146.5 171) (end 146.5 254.5) (layer Edge.Cuts) (width 0.05))
-  (gr_line (start 160.5 171) (end 160.5 254.5) (layer Edge.Cuts) (width 0.05))
+  (gr_arc (start 162 149) (end 160.5 149) (angle -180) (layer Edge.Cuts) (width 0.05))
   (gr_arc (start 78 254.5) (end 76.5 254.5) (angle -180) (layer Edge.Cuts) (width 0.05))
-  (gr_arc (start 106 254.5) (end 104.5 254.5) (angle -180) (layer Edge.Cuts) (width 0.05))
+  (gr_arc (start 62 52) (end 62 50) (angle -90) (layer Edge.Cuts) (width 0.05))
+  (gr_arc (start 178 52) (end 180 52) (angle -90) (layer Edge.Cuts) (width 0.05))
+  (gr_arc (start 178 268) (end 178 270) (angle -90) (layer Edge.Cuts) (width 0.05))
+  (gr_arc (start 62 268) (end 60 268) (angle -90) (layer Edge.Cuts) (width 0.05))
   (gr_arc (start 92 254.5) (end 90.5 254.5) (angle -180) (layer Edge.Cuts) (width 0.05))
-  (gr_arc (start 134 171) (end 135.5 171) (angle -180) (layer Edge.Cuts) (width 0.05))
-  (gr_arc (start 92 171) (end 93.5 171) (angle -180) (layer Edge.Cuts) (width 0.05))
-  (gr_arc (start 134 254.5) (end 132.5 254.5) (angle -180) (layer Edge.Cuts) (width 0.05))
-  (gr_arc (start 148 254.5) (end 146.5 254.5) (angle -180) (layer Edge.Cuts) (width 0.05))
-  (gr_arc (start 106 171) (end 107.5 171) (angle -180) (layer Edge.Cuts) (width 0.05))
-  (gr_arc (start 162 254.5) (end 160.5 254.5) (angle -180) (layer Edge.Cuts) (width 0.05))
-  (gr_arc (start 148 171) (end 149.5 171) (angle -180) (layer Edge.Cuts) (width 0.05))
-  (gr_arc (start 120 171) (end 121.5 171) (angle -180) (layer Edge.Cuts) (width 0.05))
-  (gr_arc (start 162 171) (end 163.5 171) (angle -180) (layer Edge.Cuts) (width 0.05))
-  (gr_arc (start 120 254.5) (end 118.5 254.5) (angle -180) (layer Edge.Cuts) (width 0.05))
-  (gr_line (start 104.5 171) (end 104.5 254.5) (layer Edge.Cuts) (width 0.05))
-  (gr_line (start 163.5 171) (end 163.5 254.5) (layer Edge.Cuts) (width 0.05))
-  (gr_line (start 149.5 171) (end 149.5 254.5) (layer Edge.Cuts) (width 0.05))
-  (gr_line (start 121.5 171) (end 121.5 254.5) (layer Edge.Cuts) (width 0.05))
-  (gr_line (start 93.5 171) (end 93.5 254.5) (layer Edge.Cuts) (width 0.05))
-  (gr_line (start 90.5 171) (end 90.5 254.5) (layer Edge.Cuts) (width 0.05))
-  (gr_line (start 135.5 171) (end 135.5 254.5) (layer Edge.Cuts) (width 0.05))
-  (gr_line (start 107.5 171) (end 107.5 254.5) (layer Edge.Cuts) (width 0.05))
-  (gr_line (start 132.5 171) (end 132.5 254.5) (layer Edge.Cuts) (width 0.05))
-  (gr_line (start 118.5 171) (end 118.5 254.5) (layer Edge.Cuts) (width 0.05))
-  (gr_line (start 76.5 171) (end 76.5 254.5) (layer Edge.Cuts) (width 0.05))
-  (gr_line (start 79.5 171) (end 79.5 254.5) (layer Edge.Cuts) (width 0.05))
   (gr_line (start 94 158) (end 104 158) (layer Edge.Cuts) (width 0.05))
   (gr_arc (start 94 160) (end 94 158) (angle -180) (layer Edge.Cuts) (width 0.05))
@@
   (gr_line (start 107.5 171) (end 107.5 254.5) (layer Edge.Cuts) (width 0.05))
   (gr_line (start 93.5 171) (end 93.5 254.5) (layer Edge.Cuts) (width 0.05))
-  (gr_arc (start 162 149) (end 160.5 149) (angle -180) (layer Edge.Cuts) (width 0.05))
   (gr_arc (start 148 149) (end 146.5 149) (angle -180) (layer Edge.Cuts) (width 0.05))
   (gr_arc (start 134 149) (end 132.5 149) (angle -180) (layer Edge.Cuts) (width 0.05))
@@
   (gr_arc (start 120 254.5) (end 118.5 254.5) (angle -180) (layer Edge.Cuts) (width 0.05))
   (gr_arc (start 106 254.5) (end 104.5 254.5) (angle -180) (layer Edge.Cuts) (width 0.05))
-  (gr_arc (start 92 254.5) (end 90.5 254.5) (angle -180) (layer Edge.Cuts) (width 0.05))
   (gr_line (start 160.5 171) (end 160.5 254.5) (layer Edge.Cuts) (width 0.05))
   (gr_line (start 146.5 171) (end 146.5 254.5) (layer Edge.Cuts) (width 0.05))
@@
   (gr_line (start 107.5 65.5) (end 107.5 149) (layer Edge.Cuts) (width 0.05))
   (gr_line (start 93.5 65.5) (end 93.5 149) (layer Edge.Cuts) (width 0.05))
-  (gr_arc (start 78 254.5) (end 76.5 254.5) (angle -180) (layer Edge.Cuts) (width 0.05))
   (gr_arc (start 78 171) (end 79.5 171) (angle -180) (layer Edge.Cuts) (width 0.05))
   (gr_line (start 76.5 171) (end 76.5 254.5) (layer Edge.Cuts) (width 0.05))
@@
   (gr_line (start 76.5 65.5) (end 76.5 149) (layer Edge.Cuts) (width 0.05))
   (gr_line (start 79.5 65.5) (end 79.5 149) (layer Edge.Cuts) (width 0.05))
-  (gr_line (start 180 270) (end 60 270) (layer Edge.Cuts) (width 0.05))
-  (gr_line (start 60 50) (end 180 50) (layer Edge.Cuts) (width 0.05))
-  (gr_line (start 180 50) (end 180 270) (layer Edge.Cuts) (width 0.05))
-  (gr_line (start 60 50) (end 60 270) (layer Edge.Cuts) (width 0.05))
+  (gr_line (start 178 270) (end 62 270) (layer Edge.Cuts) (width 0.05))
+  (gr_line (start 62 50) (end 178 50) (layer Edge.Cuts) (width 0.05))
+  (gr_line (start 180 52) (end 180 268) (layer Edge.Cuts) (width 0.05))
+  (gr_line (start 60 52) (end 60 268) (layer Edge.Cuts) (width 0.05))
 )
